Commit message: update main branch

File: src/mo_hinh/urdf/xe.urdf (robot description, URDF)
Before this commit: robot my_mecanum_robot, 11 links, 10 joints
Links:
- removed link wheel_fl_link
- removed link wheel_fr_link
- removed link wheel_rl_link
- removed link wheel_rr_link
- added link sonar_center_link, mass 0.01; collision box size=0.02 0.04 0.02; visual box size=0.02 0.04 0.02
- added link sonar_left_link, mass 0.01; collision box size=0.02 0.04 0.02; visual box size=0.02 0.04 0.02
- added link sonar_right_link, mass 0.01; collision box size=0.02 0.04 0.02; visual box size=0.02 0.04 0.02
- added link wheel_left_link, mass 0.50; collision cylinder length=0.05 radius=0.08255; visual cylinder length=0.05 radius=0.08255
- added link wheel_right_link, mass 0.50; collision cylinder length=0.05 radius=0.08255; visual cylinder length=0.05 radius=0.08255
Joints:
- removed joint wheel_fl_joint
- removed joint wheel_fr_joint
- removed joint wheel_rl_joint
- removed joint wheel_rr_joint
- added joint sonar_center_joint: type fixed, parent base_link, child sonar_center_link, origin xyz=0.30 0.0 0.05 rpy=0 0 0
- added joint sonar_left_joint: type fixed, parent base_link, child sonar_left_link, origin xyz=0.30 0.20 0.05 rpy=0 0 0.785398
- added joint sonar_right_joint: type fixed, parent base_link, child sonar_right_link, origin xyz=0.30 -0.20 0.05 rpy=0 0 -0.785398
- added joint wheel_left_joint: type continuous, parent base_link, child wheel_left_link, origin xyz=0 0.29 -0.02 rpy=-1.5708 0 0, axis 0 0 1
- added joint wheel_right_joint: type continuous, parent base_link, child wheel_right_link, origin xyz=0 -0.29 -0.02 rpy=-1.5708 0 0, axis 0 0 1
- joint base_joint: origin xyz=0 0 0.05 rpy=0 0 0 -> xyz=0 0 0.08255 rpy=0 0 0
- joint laser_joint: origin xyz=0 0 0.08 rpy=0 0 0 -> xyz=-0.12 0 0.15 rpy=0 0 0

Commit message: update gui dashboard

File: src/mo_hinh/urdf/xe.urdf (robot description, URDF)
Before this commit: robot my_diff_drive_robot, 12 links, 11 joints
Links:
- added link camera_depth_optical_frame, mass 0.0001
Joints:
- added joint camera_depth_optical_joint: type fixed, parent camera_link, child camera_depth_optical_frame, origin xyz=0 0 0 rpy=-1.5708 0 -1.5708
- joint camera_joint: origin xyz=0 0 0.265 rpy=0 -0.0873 0 -> xyz=0.30 0.15 0.335 rpy=0 0.87266 0
- joint laser_joint: origin xyz=-0.12 0 0.15 rpy=0 0 0 -> xyz=+0.05 0 0.15 rpy=0 0 0

Commit message: dachinhxong

File: src/mo_hinh/urdf/xe.urdf (robot description, URDF)
Before this commit: robot my_diff_drive_robot, 13 links, 12 joints
Links:
- link support_link: geometry collision box size=0.02 0.02 0.87; visual box size=0.02 0.02 0.87
Joints:
- joint camera_joint: origin xyz=0.30 0.15 0.335 rpy=0 0.87266 0 -> xyz=0.30 0.14 0.87 rpy=0 0.698132 0; parent support_link -> base_link
- joint support_joint: origin xyz=0.15 0 0.265 rpy=0 0 0 -> xyz=0.30 0.14 0.435 rpy=0 0 0

Commit message: updaate map

File: src/mo_hinh/urdf/xe.urdf (robot description, URDF)
Before this commit: robot my_diff_drive_robot, 13 links, 12 joints
Joints:
- joint laser_joint: origin xyz=+0.05 0 0.15 rpy=0 0 0 -> xyz=0 0 0.15 rpy=0 0 0

Commit message: hoanthanhinterfaces

File: src/mo_hinh/urdf/xe.urdf (robot description, URDF)
Before this commit: robot my_diff_drive_robot, 13 links, 12 joints
Links:
- added link caster_front_left_link, mass 0.1; collision sphere radius=0.08255; visual cylinder length=0.04 radius=0.08255
- added link caster_front_right_link, mass 0.1; collision sphere radius=0.08255; visual cylinder length=0.04 radius=0.08255
Joints:
- added joint caster_front_left_joint: type fixed, parent base_link, child caster_front_left_link, origin xyz=0.23 0.20 -0.02 rpy=0 0 0
- added joint caster_front_right_joint: type fixed, parent base_link, child caster_front_right_link, origin xyz=0.23 -0.20 -0.02 rpy=0 0 0
- joint base_joint: origin xyz=0 0 0.08255 rpy=0 0 0 -> xyz=0 0 0.10255 rpy=0 0 0

Commit message: xog backend và đã chạy mô phỏng trên gazebo

File: src/mo_hinh/urdf/xe.urdf (robot description, URDF)
Before this commit: robot my_diff_drive_robot, 15 links, 14 joints
Links:
- removed link caster_front_left_link
- removed link caster_front_right_link
- removed link sonar_center_link
- removed link sonar_left_link
- removed link sonar_right_link
- added link caster_front_link, mass 0.1; collision sphere radius=0.05; visual sphere radius=0.05
- added link caster_rear_link, mass 0.1; collision sphere radius=0.05; visual sphere radius=0.05
- link base_footprint: mass 0.0001 -> None
- link laser_link: geometry visual cylinder length=0.05 radius=0.05
Joints:
- removed joint caster_front_left_joint
- removed joint caster_front_right_joint
- removed joint sonar_center_joint
- removed joint sonar_left_joint
- removed joint sonar_right_joint
- added joint caster_front_joint: type fixed, parent base_link, child caster_front_link, origin xyz=0.22 0 -0.05255 rpy=0 0 0
- added joint caster_rear_joint: type fixed, parent base_link, child caster_rear_link, origin xyz=-0.22 0 -0.05255 rpy=0 0 0
- joint base_joint: origin xyz=0 0 0.10255 rpy=0 0 0 -> xyz=0 0 0.08255 rpy=0 0 0
- joint camera_joint: origin xyz=0.30 0.14 0.87 rpy=0 0.698132 0 -> xyz=0.25 0.14 0.87 rpy=0 0.698132 0
- joint support_joint: origin xyz=0.30 0.14 0.435 rpy=0 0 0 -> xyz=0.25 0.14 0.435 rpy=0 0 0

Commit message: ok

File: src/mo_hinh/urdf/xe.urdf (robot description, URDF)
Before this commit: robot my_diff_drive_robot, 12 links, 11 joints
Links:
- added link rear_camera_depth_optical_frame, mass 0.0001
- added link rear_camera_link, mass 0.10; collision box size=0.025 0.09 0.025; visual box size=0.025 0.09 0.025
Joints:
- added joint rear_camera_depth_optical_joint: type fixed, parent rear_camera_link, child rear_camera_depth_optical_frame, origin xyz=0 0 0 rpy=-1.5708 0 -1.5708
- added joint rear_camera_joint: type fixed, parent base_link, child rear_camera_link, origin xyz=-0.25 0.14 0.87 rpy=0 0.698132 3.14159265

Commit message: ok

File: src/mo_hinh/urdf/xe.urdf (robot description, URDF)
Before this commit: robot my_diff_drive_robot, 14 links, 13 joints
Joints:
- joint camera_joint: origin xyz=0.25 0.14 0.87 rpy=0 0.698132 0 -> xyz=0.28 0.14 0.87 rpy=0 0.698132 0
- joint rear_camera_joint: origin xyz=-0.25 0.14 0.87 rpy=0 0.698132 3.14159265 -> xyz=-0.28 0.14 0.87 rpy=0 0.698132 3.14159265

Commit message: ok

File: src/mo_hinh/urdf/xe.urdf (robot description, URDF)
Before this commit: robot my_diff_drive_robot, 14 links, 13 joints
Links:
- added link rear_scan_frame
Joints:
- added joint rear_scan_joint: type fixed, parent base_link, child rear_scan_frame, origin xyz=-0.28 0.14 0.0 rpy=0 0 3.14159265

Commit message: restore(config,mo_hinh): revert 8 selected files to backend branch state
Restore exactly four config/ files and four src/mo_hinh/ files from backend commit 52da25d3ec554b352aa62b5548c73cbeed1633c7. Preserve all other files from main unchanged.

File: src/mo_hinh/urdf/xe.urdf (robot description, URDF)
Before this commit: robot my_diff_drive_robot, 15 links, 14 joints
Links:
- removed link rear_camera_depth_optical_frame
- removed link rear_camera_link
- removed link rear_scan_frame
Joints:
- removed joint rear_camera_depth_optical_joint
- removed joint rear_camera_joint
- removed joint rear_scan_joint
- joint camera_joint: origin xyz=0.28 0.14 0.87 rpy=0 0.698132 0 -> xyz=0.25 0.14 0.87 rpy=0 0.698132 0
